File: TestPlate/HeadlessLogicTester.kicad_pcb (KiCad board)
At the start: 2 copper layers, 195.1 x 84 mm, 33 parts, among them J1 EXT_HDR, J2 Test Result Capture, J3 Test Input, U1 CD74HC4094E, U2 CD74HC4094E, U3 CD74HC4094E, U4 CD74HC4094E, U5 CD4066B, U6 74HC166, U7 74HC166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

Commit message: Readme update for rev0 sharing.
Other:
- board text added: "TestPlate"
- board text removed: "Loaf Plate Tester"
Changed lines of the file:
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@@
   (setup
     (stackup
-      (layer "F.SilkS" (type "Top Silk Screen"))
+      (layer "F.SilkS" (type "Top Silk Screen") (color "White"))
       (layer "F.Paste" (type "Top Solder Paste"))
-      (layer "F.Mask" (type "Top Solder Mask") (thickness 0.01))
+      (layer "F.Mask" (type "Top Solder Mask") (color "Black") (thickness 0.01))
       (layer "F.Cu" (type "copper") (thickness 0.035))
       (layer "dielectric 1" (type "core") (thickness 1.51) (material "FR4") (epsilon_r 4.5) (loss_tangent 0.02))
       (layer "B.Cu" (type "copper") (thickness 0.035))
-      (layer "B.Mask" (type "Bottom Solder Mask") (thickness 0.01))
+      (layer "B.Mask" (type "Bottom Solder Mask") (color "Black") (thickness 0.01))
       (layer "B.Paste" (type "Bottom Solder Paste"))
-      (layer "B.SilkS" (type "Bottom Silk Screen"))
+      (layer "B.SilkS" (type "Bottom Silk Screen") (color "White"))
       (copper_finish "HAL SnPb")
       (dielectric_constraints no)
@@
     (effects (font (size 1 1) (thickness 0.15)))
   )
-  (gr_text "Loaf\nPlate\nTester" (at 199.39 86.36) (layer "F.SilkS")
+  (gr_text "TestPlate" (at 194.564 86.36) (layer "F.SilkS")
     (effects (font (size 5 5) (thickness 0.35)) (justify left))
   )
