File: ClockPlate/ClockPlate.kicad_sch (KiCad schematic)
At the start: 48 parts

Commit message: First version of the ClockPlate schematic.
Parts:
- added C10, C11, C12, C13, C14, C15, C16, C17, C9: 0u1, Capacitor_THT:C_Rect_L4.0mm_W2.5mm_P2.50mm, symbol Device:C_Small
- added C18, C19, C20, C21, C22, C23, C24, C25, C26: 0u01, Capacitor_THT:C_Rect_L4.0mm_W2.5mm_P2.50mm, symbol Device:C_Small
- added D2: CLK_LED, LED_THT:LED_D5.0mm, symbol Device:LED
- added D3: ~{CLK}_LED, LED_THT:LED_D5.0mm, symbol Device:LED
- added J1: Signal Header, ExtraParts:LP_EXT, symbol Connector_Generic:Conn_02x05_Counter_Clockwise
- added JP1: CLK_LED_JMP, Connector_PinHeader_2.54mm:PinHeader_1x02_P2.54mm_Vertical, symbol Jumper:Jumper_2_Bridged
- added JP2: ~{CLK}_LED_JMP, Connector_PinHeader_2.54mm:PinHeader_1x02_P2.54mm_Vertical, symbol Jumper:Jumper_2_Bridged
- added R11, R12: 330, Resistor_THT:R_Axial_DIN0207_L6.3mm_D2.5mm_P10.16mm_Horizontal, symbol Device:R_Small
- added U5: SN74AC74N, Package_DIP:DIP-14_W7.62mm_Socket_LongPads, symbol ExtraParts:SN74AC74N
- added U8: SN74AC00N, Package_DIP:DIP-14_W7.62mm_Socket_LongPads, symbol ExtraParts:SN74AC00N
- C1: renamed from C?; value 10u -> 1u; footprint (none) -> Capacitor_THT:CP_Radial_D5.0mm_P2.00mm
- C2, C3, C4, C5, C7, C8: renamed from C?; footprint (none) -> Capacitor_THT:C_Rect_L4.0mm_W2.5mm_P2.50mm
- C6: renamed from C?; footprint (none) -> Capacitor_THT:CP_Radial_D6.3mm_P2.50mm
- D1: renamed from D?; value Reset LED -> ~{RES}_LED; footprint (none) -> LED_THT:LED_D5.0mm
- R1, R10, R2, R3, R4, R5, R6, R7, R8, R9: renamed from R?; footprint (none) -> Resistor_THT:R_Axial_DIN0207_L6.3mm_D2.5mm_P10.16mm_Horizontal
- RV1: renamed from RV?; footprint (none) -> Potentiometer_THT:Potentiometer_Bourns_3386X_Horizontal
- RV2: renamed from RV?; footprint (none) -> Potentiometer_THT:Potentiometer_Bourns_3266W_Vertical
- SW1, SW3: renamed from SW?; footprint (none) -> Button_Switch_THT:SW_PUSH_6mm
- SW2, SW4: renamed from SW?; footprint (none) -> Button_Switch_THT:SW_E-Switch_EG1271_DPDT
- U1, U4, U9: renamed from U?; footprint Package_DIP:DIP-14_W7.62mm_LongPads -> Package_DIP:DIP-14_W7.62mm_Socket_LongPads
- U10, U3, U6, U7: renamed from U?; footprint Package_DIP:DIP-8_W7.62mm -> Package_DIP:DIP-8_W7.62mm_Socket_LongPads
- U2: renamed from U?; footprint (none) -> Package_DIP:DIP-14_W7.62mm_Socket_LongPads
- gave numbers to parts that had none: 2
Connections:
- net RESB is gone; now on net ~{RES}: R6.1, R7.2, U9.2 (1Y), U9.3 (2A)
- net +5V: now also U1.17 (VCC), U2.17 (VCC), U4.14 (VCC), C10.2, C11.2, C12.2, C13.2, C14.2, C15.2, C16.2, C17.2, C18.2, C19.2, C20.2, C21.2, C22.2, C23.2, C24.2, C25.2, C26.2, C9.2, U5.1 (1~{CLR}), U5.14 (VCC), U5.4 (1~{PRE}), U8.17 (VCC)
- net GND: now also U1.7 (GND), U2.7 (GND), U4.7 (GND), C10.1, C11.1, C12.1, C13.1, C14.1, C15.1, C16.1, C17.1, C18.1, C19.1, C20.1, C21.1, C22.1, C23.1, C24.1, C25.1, C26.1, C9.1, D2.1 (K), D3.1 (K), U5.10 (2~{PRE}), U5.11 (2CLK), U5.12 (2D), U5.13 (2~{CLR}), U5.7 (GND), U8.10 (3B), U8.12 (4A), U8.13 (4B), U8.7 (GND), U8.9 (3A)
- net HLT: now also PLT1.9 (IO3), J1.5 (Pin_5), J1.6 (Pin_6)
- net RES: now also PLT1.8 (IO5), J1.3 (Pin_3), J1.8 (Pin_8)
- net at SW4.2 (B): now also U5.3 (1CLK)
- net ~{RES}: now reaches PLT1.10 (IO4)
- net ~{RES}: now also J1.4 (Pin_4), J1.7 (Pin_7)
- net CLK: now reaches PLT1.5 (IO1)
- net CLK: now also J1.1 (Pin_1), J1.10 (Pin_10), JP1.1 (A), U8.6 (2Y)
- net ~{CLK}: now reaches PLT1.7 (IO2)
- net ~{CLK}: now also J1.2 (Pin_2), J1.9 (Pin_9), JP2.1 (A), U8.3 (1Y)
- new net: U5.5 (1Q), U8.1 (1A), U8.2 (1B)
- new net: JP2.2 (B), R12.1
- new net: D3.2 (A), R12.2
- new net: JP1.2 (B), R11.1
- new net: D2.2 (A), R11.2
- new net: U5.2 (1D), U5.6 (1~{Q}), U8.4 (2A), U8.5 (2B)
- no-connect marks 18 -> 17
Other:
- moved on the sheet: C1, C2, C3, C4, C5, C6, C7, C8, D1, PLT1, R1, R2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

Commit message: Completed Rev0 of ClockPlate
Parts:
- added J2: Signal Header, Connector_PinSocket_2.54mm:PinSocket_2x05_P2.54mm_Vertical, symbol Connector_Generic:Conn_02x05_Odd_Even
- C1: Manufacturer Name (none) -> Würth Elektronik; Manufacturer Part Number (none) -> 860020772005; Supplier Name (none) -> Digi-Key; Supplier Part Number (none) -> 732-8966-1-ND
- C10, C11, C12, C13, C14, C15, C16, C17, C3, C8, C9: Manufacturer Name (none) -> Vishay Beyschlag/Draloric/BC Components; Manufacturer Part Number (none) -> K104Z15Y5VE5TL2; Supplier Name (none) -> Digi-Key; Supplier Part Number (none) -> BC1148CT-ND
- C18, C19, C2, C20, C21, C22, C23, C24, C25, C26, C4, C5, C7: Manufacturer Name (none) -> KEMET; Manufacturer Part Number (none) -> C315C103J3G5TA; Supplier Name (none) -> Digi-Key; Supplier Part Number (none) -> C315C103J3G5TA-ND
- C6: Manufacturer Name (none) -> Würth Elektronik; Manufacturer Part Number (none) -> 870055673001; Supplier Name (none) -> Digi-Key; Supplier Part Number (none) -> 732-6367-1-ND
- D1, D3: Manufacturer Name (none) -> SunLED; Manufacturer Part Number (none) -> XSDG23MB; Supplier Name (none) -> Digi-Key; Supplier Part Number (none) -> 1497-1042-ND
- D2: Manufacturer Name (none) -> SunLED; Manufacturer Part Number (none) -> XSCBD23MB; Supplier Name (none) -> Digi-Key; Supplier Part Number (none) -> 1497-1037-ND
- J1: symbol Connector_Generic:Conn_02x05_Counter_Clockwise -> Connector_Generic:Conn_02x05_Odd_Even; Manufacturer Name (none) -> On Shore Technology Inc.; Manufacturer Part Number (none) -> 302-R101; Supplier Name (none) -> Digi-Key; Supplier Part Number (none) -> ED10533-ND
- JP1, JP2: Manufacturer Name (none) -> Amphenol ICC (FCI); Manufacturer Part Number (none) -> 68000-102HLF; Supplier Name (none) -> Digi-Key; Supplier Part Number (none) -> 609-3500-ND
- PLT1: footprint CustomFootprintLibrary:Breadboard_Busx02_Terminalx01_Tiesx830_WithMounts -> ExtraParts:BasePlate with Extension; Manufacturer Name (none) -> JLCPCB; Supplier Name (none) -> JLCPCB
- R1, R2, R4, R5, R7, R8: Manufacturer Name (none) -> TE Connectivity Passive Product; Manufacturer Part Number (none) -> YR1B1K0CC; Supplier Name (none) -> Digi-Key; Supplier Part Number (none) -> A105942CT-ND
- R10, R6: Manufacturer Name (none) -> YAGEO; Manufacturer Part Number (none) -> MFP-25BRD52-3K3; Supplier Name (none) -> Digi-Key; Supplier Part Number (none) -> 3.3KADCT-ND
- R11, R12: Manufacturer Name (none) -> TE Connectivity Passive Product; Manufacturer Part Number (none) -> CFR16J330R; Supplier Name (none) -> Digi-Key; Supplier Part Number (none) -> A129436CT-ND
- R3, R9: Manufacturer Name (none) -> TE Connectivity Passive Product; Manufacturer Part Number (none) -> YR1B1M0CC; Supplier Name (none) -> Digi-Key; Supplier Part Number (none) -> A105943CT-ND
- RV1: Manufacturer Name (none) -> Bourns Inc.; Manufacturer Part Number (none) -> 3386X-1-105TLF; Supplier Name (none) -> Digi-Key; Supplier Part Number (none) -> 3386X-1-105TLF-ND
- RV2: Manufacturer Name (none) -> Bourns Inc.; Manufacturer Part Number (none) -> 3266W-1-204LF; Supplier Name (none) -> Digi-Key; Supplier Part Number (none) -> 3266W-204LF-ND
- SW1, SW3: Manufacturer Name (none) -> Omron Electronics Inc-EMC Div; Manufacturer Part Number (none) -> B3F-1002; Supplier Name (none) -> Digi-Key; Supplier Part Number (none) -> SW401-ND
- SW2: Manufacturer Name (none) -> E-Switch; Manufacturer Part Number (none) -> EG1271; Supplier Name (none) -> Digi-Key; Supplier Part Number (none) -> EG1918-ND
- SW4: symbol Switch:SW_SPDT -> Switch:SW_Push_DPDT; Manufacturer Name (none) -> E-Switch; Manufacturer Part Number (none) -> EG1271; Supplier Name (none) -> Digi-Key; Supplier Part Number (none) -> EG1918-ND
- U1: Manufacturer Name (none) -> Texas Instruments; Manufacturer Part Number (none) -> SN74AC32N; Supplier Name (none) -> Digi-Key; Supplier Part Number (none) -> 296-4318-5-ND
- U10, U3, U6, U7: Manufacturer Name (none) -> Texas Instruments; Manufacturer Part Number (none) -> NE555P; Supplier Name (none) -> Digi-Key; Supplier Part Number (none) -> 296-NE555P-ND
- U2: Manufacturer Name (none) -> Texas Instruments; Manufacturer Part Number (none) -> SN74AC08N; Supplier Name (none) -> Digi-Key; Supplier Part Number (none) -> 296-33637-5-ND
- U4: Manufacturer Name (none) -> Texas Instruments; Manufacturer Part Number (none) -> SN74AC04N; Supplier Name (none) -> Digi-Key; Supplier Part Number (none) -> 296-4290-5-ND
- U4: renamed from U9; value 74AC04N_Multi -> SN74AC04N_Multi; symbol ExtraParts:74AC04N_Multi -> ExtraParts:SN74AC04N_Multi; Manufacturer Name (none) -> Texas Instruments; Manufacturer Part Number (none) -> SN74AC04N; Supplier Name (none) -> Digi-Key; Supplier Part Number (none) -> 296-4290-5-ND
- U5: Manufacturer Name (none) -> Texas Instruments; Manufacturer Part Number (none) -> SN74AC74N; Supplier Name (none) -> Digi-Key; Supplier Part Number (none) -> 296-4342-5-ND
- U8: Manufacturer Name (none) -> Texas Instruments; Manufacturer Part Number (none) -> SN74AC00N; Supplier Name (none) -> Digi-Key; Supplier Part Number (none) -> 296-4287-5-ND
Connections:
- net +5V: now also U1.14 (VCC), U2.14 (VCC), U8.14 (VCC); no longer U1.17 (VCC), U2.17 (VCC), U8.17 (VCC)
- net CLK: now also J1.2 (Pin_2), J2.1 (Pin_1), J2.2 (Pin_2); no longer J1.10 (Pin_10), PLT1.5 (IO1)
- net CLK_FAST: now also SW4.6 (C)
- net CLK_SLOW: now also SW4.4 (A)
- net HLT: now also J1.10 (Pin_10), J1.9 (Pin_9), J2.10 (Pin_10), J2.9 (Pin_9); no longer J1.5 (Pin_5), J1.6 (Pin_6), PLT1.9 (IO3)
- net RES: now also J1.5 (Pin_5), J1.6 (Pin_6), J2.5 (Pin_5), J2.6 (Pin_6); no longer J1.3 (Pin_3), J1.8 (Pin_8), PLT1.8 (IO5)
- net ~{CLK}: now also J1.3 (Pin_3), J1.4 (Pin_4), J2.3 (Pin_3), J2.4 (Pin_4); no longer J1.2 (Pin_2), J1.9 (Pin_9), PLT1.7 (IO2)
- net ~{RES}: now also J1.8 (Pin_8), J2.7 (Pin_7), J2.8 (Pin_8); no longer J1.4 (Pin_4), PLT1.10 (IO4)
- net CLK_SEL: now reaches SW4.2 (B), U5.3 (1CLK)
- net CLK_SEL: now also SW4.5 (B)
- no-connect marks 17 -> 22
Other:
- moved on the sheet: X1
